File: audio.brd (EAGLE design)
At the start: 64.8 x 36.8 mm, 42 parts, among them CN1 PH-1X06SG, CN2 PH-1X06RG, CN3 STEREO-3.5-MJ8435, CN4 STEREO-3.5-MJ8435, CN5 DC-JACK-18742, IC1 R5F104BCAFP, IC2 NJM2746E, IC3 NJM2746E, IC4 VBT1-S5-S5-SMT, IC5 NJM2866F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

Commit message: Reworked everything
Parts:
- removed IC3: NJM2746E, MyLib:EMP8
- removed R10, R7: 10k, MyLib:R2012
- C7, C8: value 0.1u -> (none)
- R3, R6: value 10k -> (none)
- moved C8 59.6 mm to (1.27, -22.9), flipped to the top
- moved R6 52.0 mm to (1.27, -11.4), flipped to the top
- moved C7 51.8 mm to (1.27, -17.1), flipped to the top
- moved R3 45.0 mm to (1.27, -5.71), flipped to the top
Connections:
- removed net N$1: IC2.P$1, IC2.P$2, R4.1, R5.1
- removed net N$12: IC3.P$3, R10.2, R7.1
- removed net N$6: IC2.P$3, R3.1, R6.2
- new net V+: IC2.P$8
- new net V-: IC2.P$4
- net +3V3: no longer C7.1, C8.1, IC2.P$8, IC3.P$8, R3.2, R7.2
- net GND: no longer C7.2, C8.2, IC2.P$4, IC3.P$4, R10.1, R6.1
- net N$11: no longer IC3.P$1, IC3.P$2, R9.1
- net N$13: now also IC2.P$3; no longer IC3.P$5
- net N$14: now also IC2.P$2; no longer IC3.P$6
- net N$16: now also IC2.P$1; no longer IC3.P$7
Routing:
- net N$1: track 10.1 -> 0.00 mm
- net N$6: track 8.52 -> 0.00 mm
- net N$12: track 8.52 -> 0.00 mm
- net +3V3: track 8.49 -> 0.00 mm
- net N$11: track 11.2 -> 6.57 mm
- net N$14: track 8.11 -> 4.64 mm
- net N$16: track 2.91 -> 0.48 mm
- net N$13: track 2.94 -> 1.58 mm
Changed lines of the file:
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@@
 <element name="C3" library="MyLib" package="C2012" value="10u" x="17.4625" y="26.67" rot="MR0"/>
 <element name="C4" library="MyLib" package="C2012" value="10u" x="3.175" y="26.3525" rot="MR0"/>
-<element name="R3" library="MyLib" package="R2012" value="10k" x="21.2725" y="34.6075" rot="MR0"/>
 <element name="R4" library="MyLib" package="R2012" value="10k" x="21.9075" y="26.67" rot="MR0"/>
 <element name="R5" library="MyLib" package="R2012" value="10k" x="26.035" y="26.67" rot="MR180"/>
-<element name="R6" library="MyLib" package="R2012" value="10k" x="25.4" y="34.6075" rot="MR0"/>
 <element name="C5" library="MyLib" package="C2012" value="1u" x="3.81" y="22.86" rot="MR0"/>
 <element name="C6" library="MyLib" package="C2012" value="1u" x="3.81" y="19.3675" rot="MR0"/>
-<element name="IC3" library="MyLib" package="EMP8" value="NJM2746E" x="7.9375" y="30.7975" rot="MR0"/>
-<element name="R7" library="MyLib" package="R2012" value="10k" x="7.3025" y="34.6075" rot="MR0"/>
 <element name="R8" library="MyLib" package="R2012" value="10k" x="11.43" y="26.3525" rot="MR180"/>
 <element name="R9" library="MyLib" package="R2012" value="10k" x="7.3025" y="26.3525" rot="MR0"/>
-<element name="R10" library="MyLib" package="R2012" value="10k" x="11.43" y="34.6075" rot="MR0"/>
-<element name="C7" library="MyLib" package="C2012" value="0.1u" x="3.175" y="34.6075" rot="MR0"/>
-<element name="C8" library="MyLib" package="C2012" value="0.1u" x="17.145" y="34.6075" rot="MR0"/>
 <element name="R11" library="MyLib" package="R2012" value="10k" x="16.51" y="30.7975" rot="MR90"/>
 <element name="R12" library="MyLib" package="R2012" value="10k" x="2.2225" y="30.7975" rot="MR90"/>
@@
 <element name="C9" library="MyLib" package="C2012" value="0.1u" x="54.9275" y="29.21" rot="MR0"/>
 <element name="R19" library="MyLib" package="R2012" value="4.7k" x="59.69" y="17.4625" rot="MR270"/>
+<element name="R3" library="MyLib" package="R2012" value="" x="1.27" y="-5.715"/>
+<element name="R6" library="MyLib" package="R2012" value="" x="1.27" y="-11.43"/>
+<element name="C7" library="MyLib" package="C2012" value="" x="1.27" y="-17.145"/>
+<element name="C8" library="MyLib" package="C2012" value="" x="1.27" y="-22.86"/>
 </elements>
 <signals>
@@
 <contactref element="C5" pad="2"/>
 <contactref element="C6" pad="2"/>
-<contactref element="IC2" pad="P$4"/>
-<contactref element="IC3" pad="P$4"/>
-<contactref element="R6" pad="1"/>
-<contactref element="R10" pad="1"/>
 <contactref element="CN3" pad="1"/>
 <contactref element="CN4" pad="1"/>
-<contactref element="C7" pad="2"/>
-<contactref element="C8" pad="2"/>
 <contactref element="U$3" pad="P$2"/>
 <contactref element="U$2" pad="P$3"/>
@@
 <contactref element="IC5" pad="P$5"/>
 <contactref element="C6" pad="1"/>
-<contactref element="IC2" pad="P$8"/>
-<contactref element="R3" pad="2"/>
-<contactref element="IC3" pad="P$8"/>
-<contactref element="R7" pad="2"/>
-<contactref element="C7" pad="1"/>
-<contactref element="C8" pad="1"/>
 <contactref element="R13" pad="1"/>
-<wire x1="20.2955" y1="34.6075" x2="19.05" y2="34.6075" width="0.4064" layer="16"/>
-<wire x1="19.05" y1="34.6075" x2="17.995" y2="34.6075" width="0.4064" layer="16"/>
-<wire x1="18.9575" y1="32.7025" x2="18.9575" y2="34.515" width="0.4064" layer="16"/>
-<wire x1="18.9575" y1="34.515" x2="19.05" y2="34.6075" width="0.4064" layer="16"/>
-<wire x1="4.025" y1="34.6075" x2="5.08" y2="34.6075" width="0.4064" layer="16"/>
-<wire x1="5.08" y1="34.6075" x2="6.3255" y2="34.6075" width="0.4064" layer="16"/>
-<wire x1="4.9875" y1="32.7025" x2="4.9875" y2="34.515" width="0.4064" layer="16"/>
-<wire x1="4.9875" y1="34.515" x2="5.08" y2="34.6075" width="0.4064" layer="16"/>
-<wire x1="20.2955" y1="34.6075" x2="44.4255" y2="17.78" width="0" layer="19" extent="16-16"/>
-<wire x1="6.3255" y1="34.6075" x2="17.995" y2="34.6075" width="0" layer="19" extent="16-16"/>
-<wire x1="9.0775" y1="22.8575" x2="4.9875" y2="32.7025" width="0" layer="19" extent="16-16"/>
-<wire x1="4.66" y1="19.3675" x2="9.0775" y2="22.8575" width="0" layer="19" extent="16-16"/>
-<wire x1="10.16" y1="16.217" x2="4.66" y2="19.3675" width="0" layer="19" extent="16-16"/>
-<wire x1="12.407" y1="11.43" x2="10.16" y2="16.217" width="0" layer="19" extent="16-16"/>
-<wire x1="14.98" y1="12.01" x2="12.407" y2="11.43" width="0" layer="19" extent="16-16"/>
+<wire x1="14.98" y1="12.01" x2="44.4255" y2="17.78" width="0" layer="19" extent="16-16"/>
+<wire x1="12.407" y1="11.43" x2="14.98" y2="12.01" width="0" layer="19" extent="16-16"/>
+<wire x1="10.16" y1="16.217" x2="12.407" y2="11.43" width="0" layer="19" extent="16-16"/>
+<wire x1="4.66" y1="19.3675" x2="10.16" y2="16.217" width="0" layer="19" extent="16-16"/>
+<wire x1="9.0775" y1="22.8575" x2="4.66" y2="19.3675" width="0" layer="19" extent="16-16"/>
 <wire x1="7.2" y1="7.62" x2="12.407" y2="11.43" width="0" layer="19" extent="16-16"/>
 </signal>
@@
 </polygon>
 </signal>
-<signal name="N$1">
-<contactref element="IC2" pad="P$1"/>
-<contactref element="R4" pad="1"/>
-<contactref element="IC2" pad="P$2"/>
-<contactref element="R5" pad="1"/>
-<wire x1="24.8575" y1="32.7025" x2="24.8575" y2="31.4325" width="0.4064" layer="16"/>
-<wire x1="22.8845" y1="26.67" x2="25.058" y2="26.67" width="0.4064" layer="16"/>
-<wire x1="25.058" y1="26.67" x2="25.0825" y2="26.67" width="0.4064" layer="16"/>
-<wire x1="25.0825" y1="26.67" x2="26.3525" y2="27.94" width="0.4064" layer="16"/>
-<wire x1="26.3525" y1="27.94" x2="26.3525" y2="31.115" width="0.4064" layer="16"/>
-<wire x1="26.3525" y1="31.115" x2="26.035" y2="31.4325" width="0.4064" layer="16"/>
-<wire x1="26.035" y1="31.4325" x2="24.8575" y2="31.4325" width="0.4064" layer="16"/>
-</signal>
-<signal name="N$6">
-<contactref element="R3" pad="1"/>
-<contactref element="R6" pad="2"/>
-<contactref element="IC2" pad="P$3"/>
-<wire x1="22.2495" y1="34.6075" x2="24.423" y2="34.6075" width="0.4064" layer="16"/>
-<wire x1="24.8575" y1="30.1625" x2="23.495" y2="30.1625" width="0.4064" layer="16"/>
-<wire x1="23.495" y1="30.1625" x2="22.225" y2="31.4325" width="0.4064" layer="16"/>
-<wire x1="22.225" y1="31.4325" x2="22.225" y2="34.583" width="0.4064" layer="16"/>
-<wire x1="22.225" y1="34.583" x2="22.2495" y2="34.6075" width="0.4064" layer="16"/>
-</signal>
-<signal name="N$12">
-<contactref element="R7" pad="1"/>
-<contactref element="R10" pad="2"/>
-<contactref element="IC3" pad="P$3"/>
-<wire x1="8.2795" y1="34.6075" x2="10.453" y2="34.6075" width="0.4064" layer="16"/>
-<wire x1="10.8875" y1="30.1625" x2="9.525" y2="30.1625" width="0.4064" layer="16"/>
-<wire x1="9.525" y1="30.1625" x2="8.255" y2="31.4325" width="0.4064" layer="16"/>
-<wire x1="8.255" y1="31.4325" x2="8.255" y2="34.583" width="0.4064" layer="16"/>
-<wire x1="8.255" y1="34.583" x2="8.2795" y2="34.6075" width="0.4064" layer="16"/>
-</signal>
 <signal name="N$13">
-<contactref element="IC3" pad="P$5"/>
 <contactref element="R8" pad="2"/>
 <contactref element="C4" pad="1"/>
 <wire x1="4.025" y1="26.3525" x2="4.025" y2="27.93" width="0.4064" layer="16"/>
-<wire x1="4.025" y1="27.93" x2="4.9875" y2="28.8925" width="0.4064" layer="16"/>
-<wire x1="4.9875" y1="28.8925" x2="12.407" y2="26.3525" width="0" layer="19" extent="16-16"/>
+<contactref element="IC2" pad="P$3"/>
+<wire x1="12.407" y1="26.3525" x2="24.8575" y2="30.1625" width="0" layer="19" extent="16-16"/>
+<wire x1="4.025" y1="26.3525" x2="12.407" y2="26.3525" width="0" layer="19" extent="16-16"/>
 </signal>
 <signal name="N$11">
-<contactref element="IC3" pad="P$2"/>
-<contactref element="IC3" pad="P$1"/>
 <contactref element="R8" pad="1"/>
-<contactref element="R9" pad="1"/>
-<wire x1="8.2795" y1="26.3525" x2="10.453" y2="26.3525" width="0.4064" layer="16"/>
-<wire x1="10.8875" y1="32.7025" x2="10.8875" y2="31.4325" width="0.4064" layer="16"/>
-<wire x1="10.8875" y1="31.4325" x2="12.065" y2="31.4325" width="0.4064" layer="16"/>
 <wire x1="12.065" y1="31.4325" x2="12.3825" y2="31.115" width="0.4064" layer="16"/>
 <wire x1="12.3825" y1="31.115" x2="12.3825" y2="27.94" width="0.4064" layer="16"/>
@@
 </signal>
 <signal name="N$14">
-<contactref element="IC3" pad="P$6"/>
 <contactref element="R9" pad="2"/>
 <contactref element="R12" pad="1"/>
-<wire x1="4.9875" y1="30.1625" x2="2.5645" y2="30.1625" width="0.4064" layer="16"/>
 <wire x1="2.5645" y1="30.1625" x2="2.2225" y2="29.8205" width="0.4064" layer="16"/>
 <wire x1="6.3255" y1="26.3525" x2="6.3255" y2="27.598" width="0.4064" layer="16"/>
@@
 <wire x1="6.6675" y1="28.2575" x2="6.6675" y2="29.5275" width="0.4064" layer="16"/>
 <wire x1="6.6675" y1="29.5275" x2="6.0325" y2="30.1625" width="0.4064" layer="16"/>
-<wire x1="6.0325" y1="30.1625" x2="4.9875" y2="30.1625" width="0.4064" layer="16"/>
+<contactref element="IC2" pad="P$2"/>
+<wire x1="6.6675" y1="29.5275" x2="24.8575" y2="31.4325" width="0" layer="19" extent="16-16"/>
+<wire x1="2.5645" y1="30.1625" x2="6.0325" y2="30.1625" width="0" layer="19" extent="16-16"/>
 </signal>
 <signal name="N$16">
-<contactref element="IC3" pad="P$7"/>
 <contactref element="R12" pad="2"/>
 <contactref element="IC1" pad="29"/>
-<wire x1="4.9875" y1="31.4325" x2="2.5645" y2="31.4325" width="0.4064" layer="16"/>
 <wire x1="2.5645" y1="31.4325" x2="2.2225" y2="31.7745" width="0.4064" layer="16"/>
-<wire x1="4.9875" y1="31.4325" x2="22.28" y2="16.11" width="0" layer="19" extent="16-16"/>
+<contactref element="IC2" pad="P$1"/>
+<wire x1="22.28" y1="16.11" x2="24.8575" y2="32.7025" width="0" layer="19" extent="16-16"/>
+<wire x1="2.5645" y1="31.4325" x2="24.8575" y2="32.7025" width="0" layer="19" extent="16-16"/>
 </signal>
 <signal name="N$17">
@@
 <wire x1="55.4675" y1="25.075" x2="59.69" y2="22.567" width="0" layer="19" extent="16-16"/>
 </signal>
+<signal name="V+">
+<contactref element="IC2" pad="P$8"/>
+</signal>
+<signal name="V-">
+<contactref element="IC2" pad="P$4"/>
+</signal>
 </signals>
