File: audio.sch (EAGLE design)
At the start: 42 parts, among them CN1 PH-1X06SG, CN2 PH-1X06RG, CN3 STEREO-3.5-MJ8435, CN4 STEREO-3.5-MJ8435, CN5 DC-JACK-18742, IC1 R5F104BCAFP, IC2 NJM2746E, IC3 NJM2746E, IC4 VBT1-S5-S5-SMT, IC5 NJM2866F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

Commit message: Reworked everything
Parts:
- removed IC3: NJM2746E, MyLib:NJM2746E
- removed R10, R7: 10k, MyLib:R2012
- C7, C8: value 0.1u -> (none)
- R3, R6: value 10k -> (none)
Connections:
- removed net N$1: IC2G$1.-IN, IC2G$1.OUT, R4.1, R5.1
- removed net N$12: IC3G$1.+IN, R10.2, R7.1
- removed net N$6: IC2G$1.+IN, R3.1, R6.2
- net +3V3: no longer C7.1, C8.1, IC2G$1.V+, IC3G$1.V+, R3.2, R7.2
- net GND: no longer C7.2, C8.2, IC2G$1.V-, IC3G$1.V-, R10.1, R6.1
- net N$11: no longer IC3G$1.-IN, IC3G$1.OUT, R9.1
- net N$13: now also IC2G$1.+IN; no longer IC3G$2.+IN
- net N$14: now also IC2G$1.-IN; no longer IC3G$2.-IN
- net N$16: now also IC2G$1.OUT; no longer IC3G$2.OUT
Other:
- moved on the sheet: C4, C7, C8, IC2G$1, R3, R6
